File: hardware/fc/fc.kicad_sch (KiCad schematic)
At the start: 96 parts, among them J1 USB-C, J10 GPIO, J11 BUZZER, J2 ESC, J3 ELRS, J4 I2C, J5 GPS, J6 VTX, J7 CAM, J8 SWD, J9 UART, Q1 Si2319CDS, Q2 2N7002, U1 STM32F405RGT6, U2 ICM-42688-P, U3 W25Q128JVSIQ, U4 LMR33630BDDA, U5 AMS1117-3.3, U6 USBLC6-2SC6, Y1 8MHz

Commit message: FC-Hardware: vollständiges Routing, DRC sauber, JLCPCB-Fertigungsdaten
- Routing über alle vier Lagen: Handverdrahtung der kritischen Stellen
  (Abblockung, Schaltregler, USB-C/VBUS/CC, USB D+/D-, SPI-Bündel zum Gyro),
  Fanout in die Versorgungsflächen, Freerouting für die übrigen Signale,
  eigener Nachrouter (A*, mit Rip-up) für Restverbindungen
- Lage 2 durchgehend GND, Lage 3 VBAT/+5V/+3V3, außen GND-Restflächen
- DRC (KiCad 7.0.11): 0 Verstöße, 0 offene Verbindungen, 0 Footprint-Fehler;
  Platine <-> Schaltplan-Netzliste: 310 Pads, 0 Abweichungen
- GPIO4 auf PC5 verlegt (PA1 nicht entflechtbar), USB-C-Footprint mit an der
  Platinenkante gekürztem Bestückungsdruck
- Fertigung: Gerber, Excellon-Bohrdateien, ZIP, BOM und CPL im JLCPCB-Format
  (Ursprung linke untere Platinenecke)
- Doku: Schaltplan-PDF, Lagenbilder, DRC-Bericht, Routing-Kennzahlen,
  README mit unsicheren Stellen

Co-Authored-By: Claude Opus 5.5 <noreply@anthropic.com>
Claude-Session: https://claude.ai/code/session_01JZYB7PZbCVuDQ6ovPGKpbm
Parts:
- removed C19: 100nF, Capacitor_SMD:C_0402_1005Metric, symbol Device:C
- H1: value M3 GND -> M3; footprint MountingHole:MountingHole_3.2mm_M3_Pad -> MountingHole:MountingHole_3.2mm_M3; symbol Mechanical:MountingHole_Pad -> Mechanical:MountingHole; Beschreibung einzige Bohrung mit Masse -> (none)
- H2: value M3 -> M3 GND; footprint MountingHole:MountingHole_3.2mm_M3 -> MountingHole:MountingHole_3.2mm_M3_Pad; symbol Mechanical:MountingHole -> Mechanical:MountingHole_Pad; Beschreibung (none) -> einzige Bohrung mit Masse (neben dem ESC-Stecker)
- J1: footprint Connector_USB:USB_C_Receptacle_HRO_TYPE-C-31-M-12 -> fc_custom:USB_C_Receptacle_HRO_TYPE-C-31-M-12_Kante
Connections:
- net GND: now also H2.1; no longer H1.1
- net GPIO4: now also U1.25 (PC5); no longer U1.15 (PA1)
- net VBUS: no longer U6.5 (VBUS)
- net GYRO_RESV: no longer names the net of U2.2 (RESV)
- no-connect marks 15 -> 17
Other:
- moved on the sheet: C14, C20, C21, C22, C23, C25, C26, C27, C28, D1, L1, Q1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

Commit message: FC: JLCPCB-Bestückung vorbereitet (LCSC-Nummern, CPL-Drehlagen, ERC)
- scripts/lcsc.py: LCSC-Nummer für alle 71 Bauteile der Oberseite, Typ
  Basic/Preferred/Extended nach der JLCPCB-Liste vom 13.10.2026, Bestand mit
  Datum und Quelle; 11 Extended-Teile, 4 Preferred
- Stückliste getrennt: jlcpcb_bom.csv / jlcpcb_cpl.csv (Oberseite, maschinell),
  handbestueckung_unten.csv (Steckverbinder J2-J11)
- CPL mit Drehkorrektur (Tabelle JLCKicadTools) und Prüfliste mit Lage von
  Pin 1 bzw. Kathode/Pluspol je Bauteil; LGA-14 und HSOP-8 ohne Tabellenwert
- Basic statt Extended: 5-V-Rückführung 33k/8,2k (5,02 V) statt 100k/24,9k;
  R16 470 Ohm für die grüne InGaN-LED; Quarz CL 12 pF passend zu 18 pF
- Werte und LCSC-Felder in Schaltplan und Platine (sync_fields.py, Kupfer
  unverändert); DRC 0/0, Abgleich Platine/Schaltplan 0 Abweichungen
- ERC mit KiCad 9.0.3: 0 Fehler, 2 Warnungen (Flash /WP und /HOLD an 3,3 V)
- README: Bestellhinweise Economic PCBA, Extended-Liste, J2-Prüfung

Co-Authored-By: Claude Opus 5.5 <noreply@anthropic.com>
Claude-Session: https://claude.ai/code/session_01JZYB7PZbCVuDQ6ovPGKpbm
Parts:
- C1, C11, C14, C15, C16, C18, C2, C20, C24, C28, C3, C30, C32, C34, C4, C5, C7: LCSC (none) -> C1525
- C10, C17, C9: LCSC (none) -> C12530
- C12, C13: Beschreibung Lastkondensator (je nach Quarz pruefen) -> Lastkondensator fuer CL 12 pF; LCSC (none) -> C1549
- C21: LCSC (none) -> C48615113
- C22: Beschreibung Eingangs-Keramik X7R -> Eingangs-Keramik X7R (1210 wegen DC-Bias); LCSC (none) -> C17498688
- C23: LCSC (none) -> C307331
- C25, C8: LCSC (none) -> C52923
- C26, C27, C31: LCSC (none) -> C45783
- C29, C33: LCSC (none) -> C19702
- C6: LCSC (none) -> C19666
- D1: LCSC (none) -> C19077448
- D2: LCSC (none) -> C2480
- D3: LCSC (none) -> C2286
- D4: LCSC (none) -> C72038
- D5: LCSC (none) -> C72043
- D6: LCSC (none) -> C2128
- FB1: LCSC (none) -> C7509833
- J1: LCSC (none) -> C165948
- L1: LCSC (none) -> C6937839
- Q1: LCSC (none) -> C146287
- Q2: LCSC (none) -> C8545
- R1, R18, R2, R4, R7, R8: LCSC (none) -> C25744
- R10: value 100k -> 33k; LCSC (none) -> C25779
- R11: value 24.9k -> 8.2k; Beschreibung FB unten -> 5,02 V -> FB unten: 33k/8,2k -> 5,02 V; LCSC (none) -> C25924
- R12, R13: LCSC (none) -> C25905
- R14, R15, R5, R6: LCSC (none) -> C11702
- R16: value 1k -> 470R; Beschreibung Vorwiderstand -> Vorwiderstand (gruene InGaN-LED, Uf ca. 2,7 V); LCSC (none) -> C25117
- R17: LCSC (none) -> C25076
- R19, R20: LCSC (none) -> C25900
- R3: LCSC (none) -> C17168
- R9: LCSC (none) -> C25741
- U1: LCSC (none) -> C15742
- U2: LCSC (none) -> C1850418
- U3: LCSC (none) -> C97521
- U4: LCSC (none) -> C544370
- U5: LCSC (none) -> C6186
- U6: LCSC (none) -> C7519
- Y1: Beschreibung Quarz 8 MHz, CL ca. 10-12 pF -> Quarz 8 MHz, CL 12 pF; LCSC (none) -> C20617566

Commit message: FC: JST-SH-Buchsen unten, beidseitige JLCPCB-Bestückung
- Steckverbinder J3–J11 statt SMD-Stiftleisten jetzt JST-SH 1,0 mm
  (seitlich steckbar) wie J2; Randbuchsen an Nord-, West-, Ost- und
  Südkante, SWD und Piepser innen
- Versorgungspins der Buchsen per Handverdrahtung an die Flächen,
  M3/M4 fest vorverlegt; komplett neu geroutet (DRC 0/0, ERC 0 Fehler,
  Platine = Schaltplan 319 Pads)
- Fertigungsdaten für Standard-PCBA beider Seiten: BOM/CPL mit
  Unterseite (Megastar ZX-SH1.0, LCSC), Drehlagen aus Pad-Vergleich
  mit den JLC-Footprints (SOT-23 jetzt +180°, HSOP-8 +270° angenommen)
- README: Buchsenbelegung, Bestellablauf, Edge Rails, Prüfpunkte
- 3D-Ansichten und Lagenbilder erneuert

Co-Authored-By: Claude Opus 5.5 <noreply@anthropic.com>
Claude-Session: https://claude.ai/code/session_01JZYB7PZbCVuDQ6ovPGKpbm
Parts:
- J10: footprint Connector_PinHeader_2.54mm:PinHeader_1x08_P2.54mm_Vertical_SMD_Pin1Left -> Connector_JST:JST_SH_SM08B-SRSS-TB_1x08-1MP_P1.00mm_Horizontal; LCSC (none) -> C7430450
- J11: footprint Connector_PinHeader_2.54mm:PinHeader_1x02_P2.54mm_Vertical_SMD_Pin1Left -> Connector_JST:JST_SH_SM02B-SRSS-TB_1x02-1MP_P1.00mm_Horizontal; LCSC (none) -> C7430444
- J2: LCSC (none) -> C7430450
- J3, J4, J5, J6, J9: footprint Connector_PinHeader_2.54mm:PinHeader_1x04_P2.54mm_Vertical_SMD_Pin1Left -> Connector_JST:JST_SH_SM04B-SRSS-TB_1x04-1MP_P1.00mm_Horizontal; LCSC (none) -> C7430446
- J7: footprint Connector_PinHeader_2.54mm:PinHeader_1x03_P2.54mm_Vertical_SMD_Pin1Left -> Connector_JST:JST_SH_SM03B-SRSS-TB_1x03-1MP_P1.00mm_Horizontal; LCSC (none) -> C7430445
- J8: footprint Connector_PinHeader_2.54mm:PinHeader_1x05_P2.54mm_Vertical_SMD_Pin1Left -> Connector_JST:JST_SH_SM05B-SRSS-TB_1x05-1MP_P1.00mm_Horizontal; LCSC (none) -> C7430447
Changed lines of the file:
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@@
       )
     )
-    (property "Footprint" "Connector_PinHeader_2.54mm:PinHeader_1x02_P2.54mm_Vertical_SMD_Pin1Left"
+    (property "Footprint" "Connector_JST:JST_SH_SM02B-SRSS-TB_1x02-1MP_P1.00mm_Horizontal"
       (at 464.82 416.56 0)
       (effects
@@
     )
     (property "Beschreibung" "Piezo-Summer (+ / -)"
+      (at 464.82 416.56 0)
+      (effects
+        (font
+          (size 1.27 1.27)
+        ) hide
+      )
+    )
+    (property "LCSC" "C7430444"
       (at 464.82 416.56 0)
       (effects
@@
       )
     )
+    (property "LCSC" "C7430450"
+      (at 43.18 510.54 0)
+      (effects
+        (font
+          (size 1.27 1.27)
+        ) hide
+      )
+    )
     (pin "1"
     )
@@
       )
     )
-    (property "Footprint" "Connector_PinHeader_2.54mm:PinHeader_1x04_P2.54mm_Vertical_SMD_Pin1Left"
+    (property "Footprint" "Connector_JST:JST_SH_SM04B-SRSS-TB_1x04-1MP_P1.00mm_Horizontal"
       (at 139.7 505.46 0)
       (effects
@@
     )
     (property "Beschreibung" "ELRS-Empfaenger"
+      (at 139.7 505.46 0)
+      (effects
+        (font
+          (size 1.27 1.27)
+        ) hide
+      )
+    )
+    (property "LCSC" "C7430446"
       (at 139.7 505.46 0)
       (effects
@@
       )
     )
-    (property "Footprint" "Connector_PinHeader_2.54mm:PinHeader_1x04_P2.54mm_Vertical_SMD_Pin1Left"
+    (property "Footprint" "Connector_JST:JST_SH_SM04B-SRSS-TB_1x04-1MP_P1.00mm_Horizontal"
       (at 180.34 505.46 0)
       (effects
@@
     )
     (property "Beschreibung" "I2C extern"
+      (at 180.34 505.46 0)
+      (effects
+        (font
+          (size 1.27 1.27)
+        ) hide
+      )
+    )
+    (property "LCSC" "C7430446"
       (at 180.34 505.46 0)
       (effects
@@
       )
     )
-    (property "Footprint" "Connector_PinHeader_2.54mm:PinHeader_1x04_P2.54mm_Vertical_SMD_Pin1Left"
+    (property "Footprint" "Connector_JST:JST_SH_SM04B-SRSS-TB_1x04-1MP_P1.00mm_Horizontal"
       (at 223.52 505.46 0)
       (effects
@@
     )
     (property "Beschreibung" "GPS"
+      (at 223.52 505.46 0)
+      (effects
+        (font
+          (size 1.27 1.27)
+        ) hide
+      )
+    )
+    (property "LCSC" "C7430446"
       (at 223.52 505.46 0)
       (effects
@@
       )
     )
-    (property "Footprint" "Connector_PinHeader_2.54mm:PinHeader_1x04_P2.54mm_Vertical_SMD_Pin1Left"
+    (property "Footprint" "Connector_JST:JST_SH_SM04B-SRSS-TB_1x04-1MP_P1.00mm_Horizontal"
       (at 264.16 505.46 0)
       (effects
@@
     )
     (property "Beschreibung" "Videosender"
+      (at 264.16 505.46 0)
+      (effects
+        (font
+          (size 1.27 1.27)
+        ) hide
+      )
+    )
+    (property "LCSC" "C7430446"
       (at 264.16 505.46 0)
       (effects
@@
       )
     )
-    (property "Footprint" "Connector_PinHeader_2.54mm:PinHeader_1x03_P2.54mm_Vertical_SMD_Pin1Left"
+    (property "Footprint" "Connector_JST:JST_SH_SM03B-SRSS-TB_1x03-1MP_P1.00mm_Horizontal"
       (at 307.34 505.46 0)
       (effects
@@
     )
     (property "Beschreibung" "Kamera"
+      (at 307.34 505.46 0)
+      (effects
+        (font
+          (size 1.27 1.27)
+        ) hide
+      )
+    )
+    (property "LCSC" "C7430445"
       (at 307.34 505.46 0)
       (effects
@@
       )
     )
-    (property "Footprint" "Connector_PinHeader_2.54mm:PinHeader_1x05_P2.54mm_Vertical_SMD_Pin1Left"
+    (property "Footprint" "Connector_JST:JST_SH_SM05B-SRSS-TB_1x05-1MP_P1.00mm_Horizontal"
       (at 43.18 533.4 0)
       (effects
@@
     )
     (property "Beschreibung" "SWD"
+      (at 43.18 533.4 0)
+      (effects
+        (font
+          (size 1.27 1.27)
+        ) hide
+      )
+    )
+    (property "LCSC" "C7430447"
       (at 43.18 533.4 0)
       (effects
@@
       )
     )
-    (property "Footprint" "Connector_PinHeader_2.54mm:PinHeader_1x04_P2.54mm_Vertical_SMD_Pin1Left"
+    (property "Footprint" "Connector_JST:JST_SH_SM04B-SRSS-TB_1x04-1MP_P1.00mm_Horizontal"
       (at 83.82 530.86 0)
       (effects
@@
     )
     (property "Beschreibung" "Debug-UART"
+      (at 83.82 530.86 0)
+      (effects
+        (font
+          (size 1.27 1.27)
+        ) hide
+      )
+    )
+    (property "LCSC" "C7430446"
       (at 83.82 530.86 0)
       (effects
@@
       )
     )
-    (property "Footprint" "Connector_PinHeader_2.54mm:PinHeader_1x08_P2.54mm_Vertical_SMD_Pin1Left"
+    (property "Footprint" "Connector_JST:JST_SH_SM08B-SRSS-TB_1x08-1MP_P1.00mm_Horizontal"
       (at 127 535.94 0)
       (effects
@@
       (at 127 535.94 0)
       (effects
+        (font
+          (size 1.27 1.27)
+        ) hide
+      )
+    )
+    (property "LCSC" "C7430450"
+      (at 127 535.94 0)
+      (effects

Commit message: FC: ELRS/GPS/I²C oben, Prüfbefunde behoben, 39 Teilenummern
- ELRS, I²C und GPS als JST-SH-Buchsen oben an der Westkante (im
  verschraubten Stack steckbar); LEDs östlich des Gyros, Fiducials
  versetzt; SWD und Piepser unten an die frei gewordenen Randplätze
- Prüfbefunde: C22 mit Masse direkt an PGND des LMR33630, Akku-Pfad
  0,8 mm mit je zwei Vias, VBAT-Streifen auf Lage 3 >= 2,5 mm, C7 direkt
  an VDDA, D1 weiter von der Kante, JP2 weg von der Massebohrung, UART-
  Buchse weg von den Wärmevias, Bestückungsdruck >= 1,0 mm / 0,16 mm
- Teilenummern 43 -> 39 (100 nF alle 50 V, 10 µF/25 V, 1 k, 5,1 k),
  Akkuteiler 100k/10k, Piepser-FET AO3400A
- route: Stichleitungen über ein Pad hinaus werden mit entfernt
- Außenkontur für den Rahmen (scripts/kontur.py, docs/fc_aussenkontur.txt)
- J2 (ESC) passt noch nicht zum UAngel-ESC und wird nach der Messung
  des Nutzers umgebaut – vorher nicht bestellen

DRC 0/0, ERC 0 Fehler, Platine = Schaltplan (319 Pads)

Co-Authored-By: Claude Opus 5.5 <noreply@anthropic.com>
Claude-Session: https://claude.ai/code/session_01JZYB7PZbCVuDQ6ovPGKpbm
Parts:
- C1, C11, C14, C15, C16, C18, C2, C20, C24, C28, C3, C30, C32, C34, C4, C5, C7: LCSC C1525 -> C307331
- C29, C33: value 10uF -> 10uF/25V; LCSC C19702 -> C96446
- C6: value 4.7uF -> 10uF/25V; Beschreibung VDD Eingang, Keramik -> VDD Eingang, Keramik (gleiches Teil wie C29/C33); LCSC C19666 -> C96446
- Q2: value 2N7002 -> AO3400A; symbol Transistor_FET:2N7002 -> Transistor_FET:AO3400A; Beschreibung Piepser-Treiber -> Piepser-Treiber (V_GS(th) max. 1,45 V: an 3,3 V sicher durc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; LCSC C8545 -> C20917
- R17: value 100R -> 1k; LCSC C25076 -> C11702
- R19, R20: value 4.7k -> 5.1k; LCSC C25900 -> C25905
- R4: value 10k -> 100k; Beschreibung Spannungsteiler oben -> Spannungsteiler oben (100k: 5 mW bei 6S statt 52 mW); LCSC C25744 -> C25741
- R5: value 1k -> 10k; Beschreibung Spannungsteiler unten -> Spannungsteiler unten (11:1 wie bisher); LCSC C11702 -> C25744
Changed lines of the file:
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@@
       )
     )
-    (property "LCSC" "C1525"
+    (property "LCSC" "C307331"
       (at 101.6 58.42 0)
       (effects
@@
       )
     )
-    (property "LCSC" "C1525"
+    (property "LCSC" "C307331"
       (at 116.84 58.42 0)
       (effects
@@
       )
     )
-    (property "LCSC" "C1525"
+    (property "LCSC" "C307331"
       (at 17.78 193.04 0)
       (effects
@@
       )
     )
-    (property "LCSC" "C1525"
+    (property "LCSC" "C307331"
       (at 35.56 193.04 0)
       (effects
@@
       )
     )
-    (property "LCSC" "C1525"
+    (property "LCSC" "C307331"
       (at 53.34 193.04 0)
       (effects
@@
       )
     )
-    (property "Value" "4.7uF"
+    (property "Value" "10uF/25V"
       (at 71.755 195.58 0)
       (effects
@@
       )
     )
-    (property "Beschreibung" "VDD Eingang, Keramik"
+    (property "Beschreibung" "VDD Eingang, Keramik (gleiches Teil wie C29/C33)"
       (at 71.12 193.04 0)
       (effects
@@
       )
     )
-    (property "LCSC" "C19666"
+    (property "LCSC" "C96446"
       (at 71.12 193.04 0)
       (effects
@@
       )
     )
-    (property "LCSC" "C1525"
+    (property "LCSC" "C307331"
       (at 86.36 193.04 0)
       (effects
@@
       )
     )
-    (property "LCSC" "C1525"
+    (property "LCSC" "C307331"
       (at 53.34 231.14 0)
       (effects
@@
       )
     )
-    (property "LCSC" "C1525"
+    (property "LCSC" "C307331"
       (at 226.06 58.42 0)
       (effects
@@
       )
     )
-    (property "LCSC" "C1525"
+    (property "LCSC" "C307331"
       (at 261.62 58.42 0)
       (effects
@@
       )
     )
-    (property "LCSC" "C1525"
+    (property "LCSC" "C307331"
       (at 365.76 58.42 0)
       (effects
@@
       )
     )
-    (property "Value" "10k"
+    (property "Value" "100k"
       (at 416.56 58.42 90)
       (effects
@@
       )
     )
-    (property "Beschreibung" "Spannungsteiler oben"
+    (property "Beschreibung" "Spannungsteiler oben (100k: 5 mW bei 6S statt 52 mW)"
       (at 416.56 58.42 0)
       (effects
@@
       )
     )
-    (property "LCSC" "C25744"
+    (property "LCSC" "C25741"
       (at 416.56 58.42 0)
       (effects
@@
       )
     )
-    (property "Value" "1k"
+    (property "Value" "10k"
       (at 434.34 53.34 90)
       (effects
@@
       )
     )
-    (property "Beschreibung" "Spannungsteiler unten"
+    (property "Beschreibung" "Spannungsteiler unten (11:1 wie bisher)"
       (at 434.34 53.34 0)
       (effects
@@
       )
     )
-    (property "LCSC" "C11702"
+    (property "LCSC" "C25744"
       (at 434.34 53.34 0)
       (effects
@@
       )
     )
-    (property "LCSC" "C1525"
+    (property "LCSC" "C307331"
       (at 452.12 53.34 0)
       (effects
@@
       )
     )
-    (property "LCSC" "C1525"
+    (property "LCSC" "C307331"
       (at 487.68 53.34 0)
       (effects
@@
       )
     )
-    (property "LCSC" "C1525"
+    (property "LCSC" "C307331"
       (at 762 53.34 0)
       (effects
@@
       )
     )
-    (property "LCSC" "C1525"
+    (property "LCSC" "C307331"
       (at 749.3 106.68 0)
       (effects
@@
       )
     )
-    (property "Value" "10uF"
+    (property "Value" "10uF/25V"
       (at 89.535 396.24 0)
       (effects
@@
       )
     )
-    (property "LCSC" "C19702"
+    (property "LCSC" "C96446"
       (at 88.9 393.7 0)
       (effects
@@
       )
     )
-    (property "LCSC" "C1525"
+    (property "LCSC" "C307331"
       (at 106.68 393.7 0)
       (effects
@@
       )
     )
-    (property "LCSC" "C1525"
+    (property "LCSC" "C307331"
       (at 139.7 393.7 0)
       (effects
@@
       )
     )
-    (property "Value" "10uF"
+    (property "Value" "10uF/25V"
       (at 272.415 459.74 0)
       (effects
@@
       )
     )
-    (property "LCSC" "C19702"
+    (property "LCSC" "C96446"
       (at 271.78 457.2 0)
       (effects
@@
       )
     )
-    (property "LCSC" "C1525"
+    (property "LCSC" "C307331"
       (at 287.02 457.2 0)
       (effects
@@
   )
   (symbol
-    (lib_id "Transistor_FET:2N7002")
+    (lib_id "Transistor_FET:AO3400A")
     (at 457.2 386.08 0)
     (unit 1)
@@
       )
     )
-    (property "Value" "2N7002"
+    (property "Value" "AO3400A"
       (at 462.28 386.08 0)
       (effects
@@
       )
     )
-    (property "Datasheet" "https://www.onsemi.com/pub/Collateral/NDS7002A-D.PDF"
+    (property "Datasheet" "http://www.aosmd.com/pdfs/datasheet/AO3400A.pdf"
       (at 462.28 389.89 0)
       (effects
@@
       )
     )
-    (property "Beschreibung" "Piepser-Treiber"
+    (property "Beschreibung" "Piepser-Treiber (V_GS(th) max. 1,45 V: an 3,3 V sicher durchgeschaltet)"
       (at 457.2 386.08 0)
       (effects
@@
       )
     )
-    (property "LCSC" "C8545"
+    (property "LCSC" "C20917"
       (at 457.2 386.08 0)
       (effects
@@
       )
     )
-    (property "Value" "100R"
+    (property "Value" "1k"
       (at 477.52 386.08 90)
       (effects
@@
       )
     )
-    (property "LCSC" "C25076"
+    (property "LCSC" "C11702"
       (at 477.52 386.08 0)
       (effects
@@
       )
     )
-    (property "Value" "4.7k"
+    (property "Value" "5.1k"
       (at 581.66 386.08 90)
       (effects
@@
       )
     )
-    (property "LCSC" "C25900"
+    (property "LCSC" "C25905"
       (at 581.66 386.08 0)
       (effects
@@
       )
     )
-    (property "Value" "4.7k"
+    (property "Value" "5.1k"
       (at 599.44 386.08 90)
       (effects
@@
       )
     )
-    (property "LCSC" "C25900"
+    (property "LCSC" "C25905"
       (at 599.44 386.08 0)
       (effects

Commit message: FC: J2 auf B-Cube 4in1, getrennte 4,5-V-Schiene, C21 47 uF, Pfeil VORNE
- J2 nach Messung am B-Cube 4in1: 1 GND, 2 VBAT, 3-6 M1-M4, 7 Strom,
  8 NC (unbeschaltet), fuer 1:1-Kabel. JP2 und ESC_5V entfernt.
  Motorpins am Prozessor unveraendert (wie Sensors/motor.c).
- +4V5 wie bei Matek: VBUS -> D2 und +5V -> D7 (SS14, Unterseite) auf
  AMS1117, ELRS und GPS. VTX, Kamera und Piepser laufen an USB nicht mit.
- C21 470 uF -> 47 uF/35 V 6,3x5,4 (C48970990), Einschaltstrom.
- Nordkante = vorn: Pfeile und VORNE im Bestueckungsdruck.
- README: Firmware-Hinweise (NOVBUSSENS, DMA-Konflikt DShot/GPS-TX/
  Debug-RX, Gyro CW270 inkl. Betaflight ab 2025.12, ADC-Pins),
  J2-Lage von oben, Pruefanleitung vor dem ersten Akku.
- Neu geroutet, Aussen-GND Mindestbreite 0,25 mm; DRC 0, ERC 0 Fehler,
  Fertigungsdaten (74 oben, 8 unten, 39 Teilenummern) und Doku neu.

Co-Authored-By: Claude Opus 5.5 <noreply@anthropic.com>
Claude-Session: https://claude.ai/code/session_01JZYB7PZbCVuDQ6ovPGKpbm
Parts:
- removed JP2: ESC_5V, Jumper:SolderJumper-2_P1.3mm_Open_RoundedPad1.0x1.5mm, symbol Jumper:SolderJumper_2_Open
- added D7: SS14, Diode_SMD:D_SMA, symbol Device:D_Schottky
- C21: value 470uF/35V -> 47uF/35V; footprint Capacitor_SMD:CP_Elec_10x10.5 -> Capacitor_SMD:CP_Elec_6.3x5.4; Beschreibung Eingangs-Elko, low ESR -> Eingangs-Elko (klein wegen Einschaltstrom; die grossen Elko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; LCSC C48615113 -> C48970990
- D2: Beschreibung USB-VBUS -> 5 V, verhindert Rueckspeisung -> USB-VBUS -> 4,5-V-Schiene, verhindert Rueckspeisung in den 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
- J2: Beschreibung ESC, JST-SH 8-polig (Pinfolge pruefen!) -> ESC B-Cube 4in1, JST-SH 8-polig (Pin 8 = NC am ESC, unbesch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
- U5: Beschreibung 3,3-V-Linearregler -> 3,3-V-Linearregler (aus der 4,5-V-Schiene)
Connections:
- net ESC_5V is gone; now on net M2: J2.4 (Pin_4)
- net +5V: now also D7.2 (A); no longer C29.1, C30.1, D2.1 (K), J3.3 (Pin_3), J5.3 (Pin_3), U5.3 (VI)
- net CURR_IN: now also J2.7 (Pin_7); no longer J2.3 (Pin_3)
- net GND: now also J2.1 (Pin_1); no longer J2.2 (Pin_2)
- net M1: now also J2.3 (Pin_3); no longer J2.5 (Pin_5)
- net M2: no longer J2.6 (Pin_6)
- net M3: now also J2.5 (Pin_5); no longer J2.7 (Pin_7)
- net M4: now also J2.6 (Pin_6); no longer J2.8 (Pin_8)
- net VBAT_IN: now also J2.2 (Pin_2); no longer J2.1 (Pin_1)
- new net +4V5: C29.1, C30.1, D2.1 (K), D7.1 (K), J3.3 (Pin_3), J5.3 (Pin_3), U5.3 (VI)
- no-connect marks 17 -> 18
Other:
- note added: "- +4V5: USB (D2) oder 5-V-Regler (D7) -> AMS1117, ELRS, GPS. +5V (VTX, Kamera, Piepser) nur aus dem Regler."
- note added: "- J2 ESC (B-Cube 4in1): 1 GND, 2 VBAT, 3-6 M1-M4, 7 Strom, 8 NC (unbeschaltet); 1:1-Kabel."
- note added: "- Pinbelegung MCU siehe README.md (verbindlich: TIM3 Motoren M1 PB0, M2 PB1, M3 PA6, M4 PA7; PA4 Strom; PC0 Akku)."
- note added: "- U2 Pin 2/3 RESV laut Referenzdesign frei, 7/10/11 an GND."
- note added: "Steckverbinder"
- note removed: "- J2 ESC: Pinfolge 1 VBAT, 2 GND, 3 CURR, 4 5V, 5-8 M1-M4 - vor dem Bestellen mit dem ESC-Kabel vergleichen!"
- note removed: "- JP2 offen: ESC-5V-Pin ist nicht mit dem FC-5V verbunden (verhindert zwei Regler gegeneinander)."
- note removed: "- Pinbelegung MCU siehe README.md (verbindlich: TIM3 Motoren PB0/PB1/PA6/PA7, PC0 Akku, PA13/PA14 SWD, PA11/PA12 USB)."
- note removed: "- U2 Pin 2/3 RESV laut Referenzdesign frei, 7/10/11 an GND. C19 an Pin 2 nur wegen der Spezifikation."
- note removed: "Steckverbinder (Unterseite)"
- moved on the sheet: C33, C34, D3, D4, D5, D6, FID1, FID2, FID3, H1, H2, H3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
